File: RF Frontend Breakout/RF Frontend Breakout.kicad_sch (KiCad schematic)
At the start: 57 parts, among them IC1 QPC1022SR, IC2 GRF5504, IC3 LHA-13LN+, IC4 QPC1022SR, J1 Conn_Coaxial, J2 Conn_Coaxial, J3 Conn_Coaxial, U1 NCS-62+

Commit message: tweaks
Parts:
- removed C12, C3: 100p, Capacitor_SMD:C_0402_1005Metric, symbol Device:C
- removed C18: 2.2n, Capacitor_SMD:C_0402_1005Metric, symbol Device:C
- added C2, C21: 100p, Capacitor_SMD:C_0402_1005Metric, symbol Device:C
- added C20: 2.2n, Capacitor_SMD:C_0402_1005Metric, symbol Device:C
- renumbered C2 to C3
Connections:
- net +5V: now also C20.1
- net GND: now also IC1.6 (EN), IC4.6 (EN), R3.2, R4.1, R8.2, R9.1, TP4.1, C2.1, C2.2, C20.2, C21.1, C21.2
Other:
- note added: "Oresat put 1.68V here - even though 1.8V is what this is supposed to be - is it just not worth finding react resistor vals to achieve 1.8?"
- note added: "R3 and R4 have labelled "DNI" in the switch datasheet. We think that we can just assign values to the resistors and ignore DNI, since we definitely need a voltage divider here - though this intuition has not been checked"
- moved on the sheet: C1, C19, C3, R3, R4, R8, R9, TP4, TP9

Commit message: tweaks to PA
Connections:
- net +5V: now also C10.1, C9.1, IC2.12 (BIAS), L4.1
- new net: IC2.13 (VCC1), L3.2
Other:
- moved on the sheet: C10, C14, C15, C9, L4, L5
