File: RF Frontend Breakout/RF Frontend Breakout.kicad_sch (KiCad schematic)
At the start: 54 parts, among them IC1 QPC1022SR, IC2 GRF5504, IC3 LHA-13LN+, IC4 QPC1022SR, J3 Conn_Coaxial, J4 Conn_01x02, J5 Conn_01x02, J6 Conn_Coaxial

Commit message: finished frontend layout!
Parts:
- renumbered C20 to C1, C9 to C10, C10 to C11, C11 to C12, C12 to C16, C16 to C17, C17 to C18, C18 to C19, C1 to C2, C19 to C20, C2 to C3, C3 to C4, C4 to C5, C5 to C6, C6 to C7, C7 to C8, C8 to C9, J6 to J1, J4 to J2, J5 to J3, J3 to J4, TP2 to TP1, TP1 to TP2
