File: Unified UHF/Unified UHF.kicad_sch (KiCad schematic)
At the start: 28 parts, among them IC6 MCP1603-330I_MC, J1 Conn_01x05, J2 Conn_01x02, J3 Conn_Coaxial, U1 AT86RF215-ZU, U3 NCS-62+, X1 TYETACSANF-26.000000

Commit message: removed lin regulator
Parts:
- removed C3, C7: 4.7 uF, Capacitor_SMD:C_0402_1005Metric, symbol Device:C
- removed D1: GREEN, LED_SMD:LED_0603_1608Metric, symbol Device:LED_Small_Filled
- removed IC6: MCP1603-330I_MC, MCP1603:MCP1603-330, symbol MCP1603:MCP1603-330I_MC
- removed J2: Conn_01x02, Connector_PinSocket_2.54mm:PinSocket_1x02_P2.54mm_Vertical, symbol Connector_Generic:Conn_01x02
- removed L1: 4.7 uH, Inductor_SMD:L_0402_1005Metric, symbol Device:L
- removed R2: 3k, Resistor_SMD:R_0603_1608Metric, symbol Device:R
- removed TP1, TP5: TestPoint, TestPoint:TestPoint_THTPad_1.5x1.5mm_Drill0.7mm, symbol Connector:TestPoint
Connections:
- no-connect marks 17 -> 14
Other:
- note removed: "+5V in"
- note removed: "GND in"
- note removed: "LINEAR REGULATOR"
- note removed: "POWER SOURCE"
- note removed: "Power indicator"
- note removed: "TODO: do we want a linear regulator on this board or should we take both 3V3 and 5V inputs from power board?"
