File: Unified UHF/Unified UHF.kicad_sch (KiCad schematic)
At the start: 81 parts, among them IC1 QPC1022SR, IC2 GRF5504, IC3 LHA-13LN+, IC4 QPC1022SR, J1 Conn_01x05, J2 Conn_01x02, J3 Conn_01x02, J4 Conn_01x01, J5 PCB.SMAFST.2H.A.HT, U1 AT86RF215-ZU, U2 NCS-62+, X1 TYETACSANF-26.000000

Commit message: small changes
Parts:
- H1, H2, H3, H4: footprint MountingHole:MountingHole_3.2mm_M3 -> MountingHole:MountingHole_3.5mm_Pad
Changed lines of the file:
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@@
 			)
 		)
-		(property "Footprint" "MountingHole:MountingHole_3.2mm_M3"
+		(property "Footprint" "MountingHole:MountingHole_3.5mm_Pad"
 			(at 250.19 275.59 0)
 			(hide yes)
@@
 			)
 		)
-		(property "Footprint" "MountingHole:MountingHole_3.2mm_M3"
+		(property "Footprint" "MountingHole:MountingHole_3.5mm_Pad"
 			(at 198.12 276.86 0)
 			(hide yes)
@@
 			)
 		)
-		(property "Footprint" "MountingHole:MountingHole_3.2mm_M3"
+		(property "Footprint" "MountingHole:MountingHole_3.5mm_Pad"
 			(at 224.79 276.86 0)
 			(hide yes)
@@
 			)
 		)
-		(property "Footprint" "MountingHole:MountingHole_3.2mm_M3"
+		(property "Footprint" "MountingHole:MountingHole_3.5mm_Pad"
 			(at 275.59 276.86 0)
 			(hide yes)

Commit message: Routed coax
Connections:
- net AVSS: no longer C3.1, C4.1, C5.1, C6.1, U1.20 (DVSS), U1.23 (DVSS), U1.24 (DVSS), U1.32 (DVSS), U1.38 (DVSS)
- new net DVSS: C3.1, C4.1, C5.1, C6.1, U1.20 (DVSS), U1.23 (DVSS), U1.24 (DVSS), U1.32 (DVSS), U1.38 (DVSS)

Commit message: fixes fixes
Parts:
- C11: value 0.8p -> 10p
Connections:
- net DVSS is gone; now on net AVSS: C3.1, C4.1, C5.1, C6.1, U1.20 (DVSS), U1.23 (DVSS), U1.24 (DVSS), U1.32 (DVSS), U1.38 (DVSS)
- net AVSS: now also C11.1, U2.6
- net at U1.9 (RFN09): now also U2.1; no longer U2.4
- net at C11.2, IC1.2 (ANT): now also TP5.1, U2.4
Other:
- moved on the sheet: C11, TP5

Commit message: before updating from schematic - as for as I know this is good
Parts:
- C19, C20, C22: value 0.1u -> 100n
- H1, H2, H3, H4: footprint MountingHole:MountingHole_3.5mm_Pad -> RF Frontend Footprints:MountingHole_3.4mm_Pad(edited from 3.5mm hole)
- TP1, TP10, TP11, TP12, TP13, TP14, TP2, TP3, TP4, TP5, TP6, TP7, TP8, TP9: footprint TestPoint:TestPoint_THTPad_1.5x1.5mm_Drill0.7mm -> TestPoint:TestPoint_Pad_D1.0mm
- U1: footprint AT86RF215:QFN48_PQ_MCH -> RF Frontend Footprints:AT86Footprint
Other:
- moved on the sheet: H1, H2, H3, H4

Commit message: done prob
Parts:
- removed R11: 10k, Resistor_SMD:R_0603_1608Metric, symbol Device:R
- removed R12: 5.6k, Resistor_SMD:R_0603_1608Metric, symbol Device:R
- removed TP10, TP11, TP12, TP13, TP14, TP8, TP9: TestPoint, TestPoint:TestPoint_Pad_D1.0mm, symbol Connector:TestPoint
- H1, H2, H3, H4: symbol Mechanical:MountingHole -> Mechanical:MountingHole_Pad
- TP7: footprint TestPoint:TestPoint_Pad_D1.0mm -> TestPoint:TestPoint_THTPad_D1.5mm_Drill0.7mm
Connections:
- net +3V3: now also TP6.1
- net +5V: now also TP5.1
- net AVSS: now also H1.1, H2.1, H3.1, H4.1, TP7.1
- net at C26.1, IC4.6 (EN): now also C14.1, IC1.6 (EN), R6.2, R7.1
- net at C11.2, IC1.2 (ANT), U2.4: no longer TP5.1
- net at FL1.2 (RF_IN), IC1.4 (RF1): no longer TP7.1
- net at FL2.6 (RF_OUT), IC1.8 (RF2): no longer TP6.1

Commit message: finally done
Parts:
- added R11: 10k, Resistor_SMD:R_0603_1608Metric, symbol Device:R
Connections:
- net +3V3: now also R11.2
- net at J1.2 (Pin_2), U1.42 (SELN): now also R11.1
Changed lines of the file:
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@@
 	)
 	(junction
+		(at 66.04 124.46)
+		(diameter 0)
+		(color 0 0 0 0)
+	)
+	(junction
 		(at 278.13 68.58)
 		(diameter 0)
@@
 	(wire
 		(pts
+			(xy 57.15 116.84) (xy 68.58 116.84)
+		)
+		(stroke
+			(width 0)
+			(type default)
+		)
+	)
+	(wire
+		(pts
 			(xy 195.58 139.7) (xy 196.85 139.7)
 		)
@@
 	(wire
 		(pts
-			(xy 57.15 116.84) (xy 68.58 116.84)
-		)
-		(stroke
-			(width 0)
-			(type default)
-		)
-	)
-	(wire
-		(pts
 			(xy 106.68 165.1) (xy 120.65 165.1)
 		)
@@
 	(wire
 		(pts
+			(xy 66.04 114.3) (xy 66.04 116.84)
+		)
+		(stroke
+			(width 0)
+			(type default)
+		)
+	)
+	(wire
+		(pts
 			(xy 201.93 134.62) (xy 207.01 134.62)
 		)
@@
 		(in_pos_files yes)
 		(dnp no)
-		(fields_autoplaced yes)
 		(property "Reference" "C2"
-			(at 60.96 110.4899 0)
+			(at 58.42 107.696 0)
 			(show_name no)
 			(do_not_autoplace no)
@@
 		)
 		(property "Value" "4.7n"
-			(at 60.96 113.0299 0)
+			(at 57.912 110.49 0)
 			(show_name no)
 			(do_not_autoplace no)
@@
 	(symbol
 		(lib_id "Device:R")
+		(at 66.04 120.65 180)
+		(unit 1)
+		(body_style 1)
+		(exclude_from_sim no)
+		(in_bom yes)
+		(on_board yes)
+		(in_pos_files yes)
+		(dnp no)
+		(property "Reference" "R11"
+			(at 63.5 120.396 90)
+			(show_name no)
+			(do_not_autoplace no)
+			(effects
+				(font
+					(size 1.27 1.27)
+				)
+				(justify left)
+			)
+		)
+		(property "Value" "10k"
+			(at 66.04 118.618 90)
+			(show_name no)
+			(do_not_autoplace no)
+			(effects
+				(font
+					(size 1.27 1.27)
+				)
+				(justify left)
+			)
+		)
+		(property "Footprint" "Resistor_SMD:R_0603_1608Metric"
+			(at 67.818 120.65 90)
+			(hide yes)
+			(show_name no)
+			(do_not_autoplace no)
+			(effects
+				(font
+					(size 1.27 1.27)
+				)
+			)
+		)
+		(property "Datasheet" ""
+			(at 66.04 120.65 0)
+			(hide yes)
+			(show_name no)
+			(do_not_autoplace no)
+			(effects
+				(font
+					(size 1.27 1.27)
+				)
+			)
+		)
+		(property "Description" "Resistor"
+			(at 66.04 120.65 0)
+			(hide yes)
+			(show_name no)
+			(do_not_autoplace no)
+			(effects
+				(font
+					(size 1.27 1.27)
+				)
+			)
+		)
+		(pin "2"
+		)
+		(pin "1"
+		)
+		(instances
+			(project "Unified UHF"
+				(path "/1be17eac-b555-466e-8bd3-43262e2e1b9c"
+					(reference "R11")
+					(unit 1)
+				)
+			)
+		)
+	)
+	(symbol
+		(lib_id "Device:R")
 		(at 193.04 156.21 90)
 		(unit 1)
@@
 					(unit 1)
 				)
+			)
+		)
+	)
+	(symbol
+		(lib_id "power:+3V3")
+		(at 66.04 114.3 0)
+		(unit 1)
+		(body_style 1)
+		(exclude_from_sim no)
+		(in_bom yes)
+		(on_board yes)
+		(in_pos_files yes)
+		(dnp no)
+		(property "Reference" "#PWR010"
+			(at 66.04 118.11 0)
+			(hide yes)
+			(show_name no)
+			(do_not_autoplace no)
+			(effects
+				(font
+					(size 1.27 1.27)
+				)
+			)
+		)
+		(property "Value" "+3V3"
+			(at 66.04 110.49 0)
+			(show_name no)
+			(do_not_autoplace no)
+			(effects
+				(font
+					(size 1.27 1.27)
+				)
+			)
+		)
+		(property "Footprint" ""
+			(at 66.04 114.3 0)
+			(hide yes)
+			(show_name no)
+			(do_not_autoplace no)
+			(effects
+				(font
+					(size 1.27 1.27)
+				)
+			)
+		)
+		(property "Datasheet" ""
+			(at 66.04 114.3 0)
+			(hide yes)
+			(show_name no)
+			(do_not_autoplace no)
+			(effects
+				(font
+					(size 1.27 1.27)
+				)
+			)
+		)
+		(property "Description" "Power symbol creates a global label with name \"+3V3\""
+			(at 66.04 114.3 0)
+			(hide yes)
+			(show_name no)
+			(do_not_autoplace no)
+			(effects
+				(font
+					(size 1.27 1.27)
+				)
+			)
+		)
+		(pin "1"
+		)
+		(instances
+			(project "Unified UHF"
+				(path "/1be17eac-b555-466e-8bd3-43262e2e1b9c"
+					(reference "#PWR010")
+					(unit 1)
+				)
