File: Unified-UHF-PCB/RF Frontend Breakout.kicad_sch (KiCad schematic)
At the start: 73 parts, among them IC1 QPC1022SR, IC2 GRF5504, IC3 LHA-13LN+, IC4 QPC1022SR, J2 Conn_01x02, J3 Conn_01x02, J4 Conn_Coaxial, J5 Conn_01x05, J6 Conn_01x02, U1 AT86RF215-ZU, U3 NCS-62+, X1 TYETACSANF-26.000000

Commit message: mounting holes + design checker fixes
Parts:
- added H1, H2, H3, H4: MountingHole, MountingHole:MountingHole_3.2mm_M3, symbol Mechanical:MountingHole

Commit message: fixed PA traces
Connections:
- net +5V: now also C10.1, C11.1, IC2.12 (BIAS), L4.1
- new net: IC2.13 (VCC1), L3.2
Changed lines of the file:
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@@
-	)
-	(junction
-		(at 307.34 163.83)
-		(diameter 0)
-		(color 0 0 0 0)
 	)
 	(junction
@@
 	(wire
 		(pts
-			(xy 307.34 163.83) (xy 317.5 163.83)
-		)
-		(stroke
-			(width 0)
-			(type default)
-		)
-	)
-	(wire
-		(pts
 			(xy 359.41 80.01) (xy 372.11 80.01)
 		)
@@
 	(wire
 		(pts
-			(xy 317.5 163.83) (xy 317.5 166.37)
-		)
-		(stroke
-			(width 0)
-			(type default)
-		)
-	)
-	(wire
-		(pts
 			(xy 68.58 127) (xy 63.5 127)
 		)
@@
 	(wire
 		(pts
+			(xy 317.5 154.94) (xy 307.34 154.94)
+		)
+		(stroke
+			(width 0)
+			(type default)
+		)
+	)
+	(wire
+		(pts
 			(xy 106.68 168.91) (xy 113.03 168.91)
 		)
@@
 		)
 		(stroke
+			(width 0)
+			(type default)
+		)
+	)
+	(wire
+		(pts
+			(xy 317.5 154.94) (xy 317.5 166.37)
+		)
+		(stroke

Commit message: fixed schematic as well
Parts:
- C2: value 100n -> 2.2n
Changed lines of the file:
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@@
 			)
 		)
-		(property "Value" "100n"
+		(property "Value" "2.2n"
 			(at 198.628 130.302 0)
 			(show_name no)
